File: X17-ESC-Adapter/_autosave-X17-ESC-Adapter.kicad_pcb (KiCad board)
At the start: 2 copper layers, 9 parts, among them J2 Power In/Out

Commit message: 10/12/24
Parts:
- moved ESC3 9.98 mm to (197.0, 87.5), turned to -90 degrees
Connections:
- ESC5 pad 5: ESC2C -> ESC2B
- ESC5 pad 6: ESC2B -> ESC2C
Routing:
- net ESC3C: track 24.3 -> 0.00 mm
- net ESC3B: track 20.4 -> 0.00 mm
- net ESC3A: track 13.5 -> 1.71 mm
- net ESC2C: track 3.77 -> 0.00 mm
- net ESC2B: track 0.00 -> 3.77 mm
- added copper zone on F.Cu, net ESC2A
- added copper zone on F.Cu, net ESC2B
- added copper zone on F.Cu, net ESC2C
Changed lines of the file:
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@@
 		)
 		(property "Value" "470 Ω"
-			(at 0 0 0)
+			(at 0 -1.5 0)
 			(unlocked yes)
 			(layer "F.Fab")
@@
 			(layers "*.Cu" "*.Mask")
 			(remove_unused_layers no)
-			(net 5 "ESC2C")
+			(net 6 "ESC2B")
 			(pinfunction "M2P2")
 			(pintype "bidirectional")
@@
 			(layers "*.Cu" "*.Mask")
 			(remove_unused_layers no)
-			(net 6 "ESC2B")
+			(net 5 "ESC2C")
 			(pinfunction "M2P3")
 			(pintype "bidirectional")
@@
 		(tags "BM08B-SRSS-TBLFSN ")
 		(property "Reference" "BM08B-SRSS-TBLFSN1"
-			(at 0 -1.4284 0)
+			(at 0 -6.4284 0)
 			(unlocked yes)
 			(layer "F.SilkS")
+			(hide yes)
 			(effects
 				(font
@@
 		)
 		(property "Value" "ESC Port"
-			(at 0 -1.4284 0)
+			(at 0 -3.4284 0)
 			(unlocked yes)
 			(layer "F.Fab")
@@
 			(layer "F.Fab")
 		)
-		(fp_text user "${REFERENCE}"
-			(at 0 -1.4284 0)
-			(unlocked yes)
-			(layer "F.Fab")
-			(effects
-				(font
-					(size 1 1)
-					(thickness 0.15)
-				)
-			)
-		)
 		(pad "1" smd rect
 			(at 3.500001 -1.4284)
@@
 		)
 		(property "Value" "RED LED"
-			(at 0 1.5936 0)
+			(at -0.05 -1.5 0)
 			(layer "F.Fab")
 			(effects
@@
 	(footprint "KiCADv6:CONN3_1824750000_WED"
 		(layer "F.Cu")
-		(at 187.0334 87.9572)
+		(at 197 87.5 -90)
 		(tags "1824750000 ")
 		(property "Reference" "ESC3"
-			(at 5 3.500001 0)
+			(at 5 3.500001 -90)
 			(unlocked yes)
 			(layer "F.SilkS")
@@
 		)
 		(property "Value" "1824750000"
-			(at 5 3.500001 0)
+			(at 5 3.500001 -90)
 			(unlocked yes)
 			(layer "F.Fab")
@@
 		)
 		(property "Footprint" "KiCADv6:CONN3_1824750000_WED"
-			(at 0 0 0)
+			(at 0 0 90)
 			(layer "F.Fab")
 			(hide yes)
@@
 		)
 		(property "Datasheet" "1824750000"
-			(at 0 0 0)
+			(at 0 0 90)
 			(layer "F.Fab")
 			(hide yes)
@@
 		)
 		(property "Description" ""
-			(at 0 0 0)
+			(at 0 0 90)
 			(layer "F.Fab")
 			(hide yes)
@@
 		)
 		(fp_line
-			(start -2.2263 -1.826999)
-			(end -2.2263 12.422401)
+			(start -2.2263 12.422401)
+			(end 12.2263 12.422401)
 			(stroke
 				(width 0.1524)
@@
 		)
 		(fp_line
-			(start -2.2263 12.422401)
-			(end 12.2263 12.422401)
+			(start 12.2263 12.422401)
+			(end 12.2263 -1.826999)
 			(stroke
 				(width 0.1524)
@@
 		)
 		(fp_line
-			(start 12.2263 -1.826999)
-			(end -2.2263 -1.826999)
+			(start -2.2263 -1.826999)
+			(end -2.2263 12.422401)
 			(stroke
 				(width 0.1524)
@@
 		)
 		(fp_line
-			(start 12.2263 12.422401)
-			(end 12.2263 -1.826999)
+			(start 12.2263 -1.826999)
+			(end -2.2263 -1.826999)
 			(stroke
 				(width 0.1524)
@@
 		)
 		(fp_line
-			(start -2.3533 -1.953999)
-			(end -2.3533 12.549401)
+			(start -2.3533 12.549401)
+			(end 12.3533 12.549401)
 			(stroke
 				(width 0.1524)
@@
 		)
 		(fp_line
-			(start -2.3533 12.549401)
-			(end 12.3533 12.549401)
+			(start 12.3533 12.549401)
+			(end 12.3533 -1.953999)
 			(stroke
 				(width 0.1524)
@@
 		)
 		(fp_line
-			(start 12.3533 -1.953999)
-			(end -2.3533 -1.953999)
+			(start -2.3533 -1.953999)
+			(end -2.3533 12.549401)
 			(stroke
 				(width 0.1524)
@@
 		)
 		(fp_line
-			(start 12.3533 12.549401)
-			(end 12.3533 -1.953999)
+			(start 12.3533 -1.953999)
+			(end -2.3533 -1.953999)
 			(stroke
 				(width 0.1524)
@@
 		)
 		(fp_line
-			(start -2.0993 -1.699999)
-			(end -2.0993 12.295401)
+			(start -2.0993 12.295401)
+			(end 12.0993 12.295401)
 			(stroke
 				(width 0.0254)
@@
 		)
 		(fp_line
-			(start -2.0993 12.295401)
-			(end 12.0993 12.295401)
+			(start 12.0993 12.295401)
+			(end 12.0993 -1.699999)
 			(stroke
 				(width 0.0254)
@@
 		)
 		(fp_line
-			(start 12.0993 -1.699999)
-			(end -2.0993 -1.699999)
+			(start -2.0993 -1.699999)
+			(end -2.0993 12.295401)
 			(stroke
 				(width 0.0254)
@@
 		)
 		(fp_line
-			(start 12.0993 12.295401)
-			(end 12.0993 -1.699999)
+			(start 12.0993 -1.699999)
+			(end -2.0993 -1.699999)
 			(stroke
 				(width 0.0254)
@@
 		)
 		(fp_text user "${REFERENCE}"
-			(at 5 3.500001 0)
+			(at 5 3.500001 -90)
 			(unlocked yes)
 			(layer "F.Fab")
@@
 		)
 		(pad "1" thru_hole circle
-			(at 0 0)
+			(at 0 0 270)
 			(size 1.7018 1.7018)
 			(drill 1.1938)
@@
 		)
 		(pad "2" thru_hole circle
-			(at 0 7.000001)
+			(at 0 7.000001 270)
 			(size 1.7018 1.7018)
 			(drill 1.1938)
@@
 		)
 		(pad "3" thru_hole circle
-			(at 5 0)
+			(at 5 0 270)
 			(size 1.7018 1.7018)
 			(drill 1.1938)
@@
 		)
 		(pad "4" thru_hole circle
-			(at 5 7.000001)
+			(at 5 7.000001 270)
 			(size 1.7018 1.7018)
 			(drill 1.1938)
@@
 		)
 		(pad "5" thru_hole circle
-			(at 10 0)
+			(at 10 0 270)
 			(size 1.7018 1.7018)
 			(drill 1.1938)
@@
 		)
 		(pad "6" thru_hole circle
-			(at 10 7.000001)
+			(at 10 7.000001 270)
 			(size 1.7018 1.7018)
 			(drill 1.1938)
@@
 		(fill none)
 		(layer "F.Cu")
+		(net 9)
 	)
 	(segment
@@
 		(width 0.2)
 		(layer "F.Cu")
-		(net 5)
+		(net 6)
 	)
 	(segment
@@
 		(width 0.2)
 		(layer "F.Cu")
-		(net 5)
-	)
-	(segment
-		(start 187.0334 94.957201)
-		(end 187.0334 87.9572)
-		(width 0.2)
-		(layer "F.Cu")
-		(net 7)
-	)
-	(segment
-		(start 187.0334 87.9572)
-		(end 182.1972 87.9572)
-		(width 0.2)
-		(layer "F.Cu")
-		(net 7)
+		(net 6)
 	)
 	(segment
@@
 	)
 	(segment
-		(start 190.490601 96.5)
-		(end 185.17 96.5)
-		(width 0.2)
-		(layer "F.Cu")
-		(net 8)
-	)
-	(segment
-		(start 185.17 96.5)
-		(end 180.99 92.32)
-		(width 0.2)
-		(layer "F.Cu")
-		(net 8)
-	)
-	(segment
-		(start 192.0334 87.9572)
-		(end 192.0334 94.957201)
-		(width 0.2)
-		(layer "F.Cu")
-		(net 8)
-	)
-	(segment
-		(start 192.0334 94.957201)
-		(end 190.490601 96.5)
-		(width 0.2)
-		(layer "F.Cu")
-		(net 8)
-	)
-	(segment
-		(start 197.0334 94.957201)
-		(end 194.100601 97.89)
-		(width 0.2)
-		(layer "F.Cu")
-		(net 9)
-	)
-	(segment
-		(start 194.100601 97.89)
-		(end 180.99 97.89)
-		(width 0.2)
-		(layer "F.Cu")
-		(net 9)
-	)
-	(segment
-		(start 197.0334 87.9572)
-		(end 197.0334 94.957201)
-		(width 0.2)
-		(layer "F.Cu")
-		(net 9)
-	)
-	(segment
 		(start 187.0334 111.122802)
 		(end 187.0334 104.122801)
@@
 			)
 		)
+	)
+	(zone
+		(net 4)
+		(net_name "ESC2A")
+		(layer "F.Cu")
+		(hatch edge 0.5)
+		(priority 4)
+		(connect_pads
+			(clearance 0.5)
+		)
+		(min_thickness 0.25)
+		(filled_areas_thickness no)
+		(fill yes
+			(thermal_gap 0.5)
+			(thermal_bridge_width 0.5)
+		)
+		(polygon
+			(pts
+				(xy 121 100.5) (xy 121 106) (xy 138 106) (xy 138 100.5)
+			)
+		)
+	)
+	(zone
+		(net 5)
+		(net_name "ESC2C")
+		(layer "F.Cu")
+		(hatch edge 0.5)
+		(priority 6)
+		(connect_pads
+			(clearance 0.5)
+		)
+		(min_thickness 0.25)
+		(filled_areas_thickness no)
+		(fill yes
+			(thermal_gap 0.5)
+			(thermal_bridge_width 0.5)
+		)
+		(polygon
+			(pts
+				(xy 121 111.5) (xy 121 117.5) (xy 138 117.5) (xy 138 111.5)
+			)
+		)
+	)
+	(zone
+		(net 6)
+		(net_name "ESC2B")
+		(layer "F.Cu")
+		(hatch edge 0.5)
+		(priority 5)
+		(connect_pads
+			(clearance 0.5)
+		)
+		(min_thickness 0.25)
+		(filled_areas_thickness no)
+		(fill yes
+			(thermal_gap 0.5)
+			(thermal_bridge_width 0.5)
+		)
+		(polygon
+			(pts
+				(xy 121 106) (xy 121 111.5) (xy 138 111.5) (xy 138 106)
+			)
+		)
