File: X17-ESC-Adapter/X17-ESC-Adapter.kicad_pcb (KiCad board)
At the start: 2 copper layers, 101.6 x 41.2 mm, 24 parts, among them J1 Pad for ESC, J10 Pad for ESC, J11 Pad for ESC, J12 Pad for ESC, J13 Pad for ESC, J2 PWM JST Connector, J3 Pad for ESC, J4 Pad for ESC, J5 Pad for ESC, J6 Pad for ESC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

Commit message: final before alumni design review
Parts:
- J1, J10, J11, J12, J13, J3, J4, J5, J6, J7, J8, J9: footprint Custom ROV Parts:Pad for ESC Adapter -> pad for esc connectors:Pad for ESC Adapter
- J2: value PWM JST Connector -> 12V Connector
- moved J5 1.18 mm to (112.5, 115.0)
- moved J1 0.50 mm to (112.5, 98.0)
- moved J3 0.29 mm to (112.5, 92.5)
- moved J7 0.23 mm to (112.5, 103.5)
- moved J6 0.14 mm to (112.5, 109.0)
Routing:
- net GND: vias 13 -> 14
Changed lines of the file:
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@@
 	(net 21 "+5V")
 	(net 22 "Current ADC")
-	(footprint "Custom ROV Parts:Pad for ESC Adapter"
+	(net 23 "unconnected-(J2-Pad01)")
+	(footprint "pad for esc connectors:Pad for ESC Adapter"
 		(layer "F.Cu")
-		(at 112.3027 92.2827)
+		(at 112.5 92.5)
 		(property "Reference" "J3"
 			(at -0.5 -4 0)
@@
 			)
 		)
-		(property "Footprint" "Custom ROV Parts:Pad for ESC Adapter"
+		(property "Footprint" "pad for esc connectors:Pad for ESC Adapter"
 			(at 0 0 0)
 			(unlocked yes)
@@
 		(pad "1" smd roundrect
 			(at 0 0 90)
-			(size 3.81 9.398)
+			(size 3.683 9.017)
 			(layers "F.Cu" "F.Paste" "F.Mask")
 			(roundrect_rratio 0.25)
@@
 		)
 	)
-	(footprint "Custom ROV Parts:Pad for ESC Adapter"
+	(footprint "pad for esc connectors:Pad for ESC Adapter"
 		(layer "F.Cu")
 		(at 203.54 104.57)
@@
 			)
 		)
-		(property "Footprint" "Custom ROV Parts:Pad for ESC Adapter"
+		(property "Footprint" "pad for esc connectors:Pad for ESC Adapter"
 			(at 0 0 0)
 			(unlocked yes)
@@
 		(pad "1" smd roundrect
 			(at 0 0 90)
-			(size 3.81 9.398)
+			(size 3.683 9.017)
 			(layers "F.Cu" "F.Paste" "F.Mask")
 			(roundrect_rratio 0.25)
@@
 		)
 	)
-	(footprint "Custom ROV Parts:Pad for ESC Adapter"
+	(footprint "pad for esc connectors:Pad for ESC Adapter"
 		(layer "F.Cu")
 		(at 203.44 98.02)
@@
 			)
 		)
-		(property "Footprint" "Custom ROV Parts:Pad for ESC Adapter"
+		(property "Footprint" "pad for esc connectors:Pad for ESC Adapter"
 			(at 0 0 0)
 			(unlocked yes)
@@
 		(pad "1" smd roundrect
 			(at 0 0 90)
-			(size 3.81 9.398)
+			(size 3.683 9.017)
 			(layers "F.Cu" "F.Paste" "F.Mask")
 			(roundrect_rratio 0.25)
@@
 			(at 0 -4.5 0)
 			(layer "F.SilkS")
+			(hide yes)
 			(effects
 				(font
@@
 			(at 0 -4.5 0)
 			(layer "F.SilkS")
+			(hide yes)
 			(effects
 				(font
@@
 			)
 		)
-		(property "Value" "PWM JST Connector"
-			(at -0.08 -3.73 0)
+		(property "Value" "12V Connector"
+			(at -0.08 -3.47 0)
 			(layer "F.Fab")
 			(effects
@@
 			(layers "*.Cu" "*.Mask")
 			(remove_unused_layers no)
+			(net 23 "unconnected-(J2-Pad01)")
 			(pinfunction "01")
 			(pintype "passive")
@@
 		)
 	)
-	(footprint "Custom ROV Parts:Pad for ESC Adapter"
+	(footprint "pad for esc connectors:Pad for ESC Adapter"
 		(layer "F.Cu")
 		(at 203.4 92.61)
@@
 			)
 		)
-		(property "Footprint" "Custom ROV Parts:Pad for ESC Adapter"
+		(property "Footprint" "pad for esc connectors:Pad for ESC Adapter"
 			(at 0 0 0)
 			(unlocked yes)
@@
 		(pad "1" smd roundrect
 			(at 0 0 90)
-			(size 3.81 9.398)
+			(size 3.683 9.017)
 			(layers "F.Cu" "F.Paste" "F.Mask")
 			(roundrect_rratio 0.25)
@@
 		)
 	)
-	(footprint "Custom ROV Parts:Pad for ESC Adapter"
+	(footprint "pad for esc connectors:Pad for ESC Adapter"
 		(layer "F.Cu")
-		(at 112.42 97.51)
+		(at 112.5 98)
 		(property "Reference" "J1"
 			(at -0.5 -4 0)
@@
 			)
 		)
-		(property "Footprint" "Custom ROV Parts:Pad for ESC Adapter"
+		(property "Footprint" "pad for esc connectors:Pad for ESC Adapter"
 			(at 0 0 0)
 			(unlocked yes)
@@
 		(pad "1" smd roundrect
 			(at 0 0 90)
-			(size 3.81 9.398)
+			(size 3.683 9.017)
 			(layers "F.Cu" "F.Paste" "F.Mask")
 			(roundrect_rratio 0.25)
@@
 			(unlocked yes)
 			(layer "F.SilkS")
+			(hide yes)
 			(effects
 				(font
@@
 			(unlocked yes)
 			(layer "F.Fab")
+			(hide yes)
 			(effects
 				(font
@@
 		)
 	)
-	(footprint "Custom ROV Parts:Pad for ESC Adapter"
+	(footprint "pad for esc connectors:Pad for ESC Adapter"
 		(layer "F.Cu")
-		(at 112.4427 113.8227)
+		(at 112.5 115)
 		(property "Reference" "J5"
-			(at 24.9727 1.2143 0)
+			(at -0.5 -4 0)
 			(unlocked yes)
 			(layer "F.SilkS")
@@
 			)
 		)
-		(property "Footprint" "Custom ROV Parts:Pad for ESC Adapter"
+		(property "Footprint" "pad for esc connectors:Pad for ESC Adapter"
 			(at 0 0 0)
 			(unlocked yes)
@@
 		(pad "1" smd roundrect
 			(at 0 0 90)
-			(size 3.81 9.398)
+			(size 3.683 9.017)
 			(layers "F.Cu" "F.Paste" "F.Mask")
 			(roundrect_rratio 0.25)
@@
 		)
 	)
-	(footprint "Custom ROV Parts:Pad for ESC Adapter"
+	(footprint "pad for esc connectors:Pad for ESC Adapter"
 		(layer "F.Cu")
 		(at 112.39 86.75)
@@
 			)
 		)
-		(property "Footprint" "Custom ROV Parts:Pad for ESC Adapter"
+		(property "Footprint" "pad for esc connectors:Pad for ESC Adapter"
 			(at 0 0 0)
 			(unlocked yes)
@@
 		(pad "1" smd roundrect
 			(at 0 0 90)
-			(size 3.81 9.398)
+			(size 3.683 9.017)
 			(layers "F.Cu" "F.Paste" "F.Mask")
 			(roundrect_rratio 0.25)
@@
 		)
 	)
-	(footprint "Custom ROV Parts:Pad for ESC Adapter"
+	(footprint "pad for esc connectors:Pad for ESC Adapter"
 		(layer "F.Cu")
-		(at 112.5027 103.7327)
+		(at 112.5 103.5)
 		(property "Reference" "J7"
 			(at -0.5 -4 0)
@@
 			)
 		)
-		(property "Footprint" "Custom ROV Parts:Pad for ESC Adapter"
+		(property "Footprint" "pad for esc connectors:Pad for ESC Adapter"
 			(at 0 0 0)
 			(unlocked yes)
@@
 		(pad "1" smd roundrect
 			(at 0 0 90)
-			(size 3.81 9.398)
+			(size 3.683 9.017)
 			(layers "F.Cu" "F.Paste" "F.Mask")
 			(roundrect_rratio 0.25)
@@
 		)
 	)
-	(footprint "Custom ROV Parts:Pad for ESC Adapter"
+	(footprint "pad for esc connectors:Pad for ESC Adapter"
 		(layer "F.Cu")
 		(at 203.59 109.89)
@@
 			)
 		)
-		(property "Footprint" "Custom ROV Parts:Pad for ESC Adapter"
+		(property "Footprint" "pad for esc connectors:Pad for ESC Adapter"
 			(at 0 0 0)
 			(unlocked yes)
@@
 		(pad "1" smd roundrect
 			(at 0 0 90)
-			(size 3.81 9.398)
+			(size 3.683 9.017)
 			(layers "F.Cu" "F.Paste" "F.Mask")
 			(roundrect_rratio 0.25)
@@
 		)
 	)
-	(footprint "Custom ROV Parts:Pad for ESC Adapter"
+	(footprint "pad for esc connectors:Pad for ESC Adapter"
 		(layer "F.Cu")
 		(at 203.53 114.7)
@@
 			)
 		)
-		(property "Footprint" "Custom ROV Parts:Pad for ESC Adapter"
+		(property "Footprint" "pad for esc connectors:Pad for ESC Adapter"
 			(at 0 0 0)
 			(unlocked yes)
@@
 		(pad "1" smd roundrect
 			(at 0 0 90)
-			(size 3.81 9.398)
+			(size 3.683 9.017)
 			(layers "F.Cu" "F.Paste" "F.Mask")
 			(roundrect_rratio 0.25)
@@
 		)
 	)
-	(footprint "Custom ROV Parts:Pad for ESC Adapter"
+	(footprint "pad for esc connectors:Pad for ESC Adapter"
 		(layer "F.Cu")
-		(at 112.5027 108.8627)
+		(at 112.5 109)
 		(property "Reference" "J6"
 			(at -0.5 -4 0)
@@
 			)
 		)
-		(property "Footprint" "Custom ROV Parts:Pad for ESC Adapter"
+		(property "Footprint" "pad for esc connectors:Pad for ESC Adapter"
 			(at 0 0 0)
 			(unlocked yes)
@@
 		(pad "1" smd roundrect
 			(at 0 0 90)
-			(size 3.81 9.398)
+			(size 3.683 9.017)
 			(layers "F.Cu" "F.Paste" "F.Mask")
 			(roundrect_rratio 0.25)
@@
 		)
 	)
-	(footprint "Custom ROV Parts:Pad for ESC Adapter"
+	(footprint "pad for esc connectors:Pad for ESC Adapter"
 		(layer "F.Cu")
 		(at 203.37 87.21)
@@
 			)
 		)
-		(property "Footprint" "Custom ROV Parts:Pad for ESC Adapter"
+		(property "Footprint" "pad for esc connectors:Pad for ESC Adapter"
 			(at 0 0 0)
 			(unlocked yes)
@@
 		(pad "1" smd roundrect
 			(at 0 0 90)
-			(size 3.81 9.398)
+			(size 3.683 9.017)
 			(layers "F.Cu" "F.Paste" "F.Mask")
 			(roundrect_rratio 0.25)
@@
 	)
 	(via
+		(at 149.5 86.5)
+		(size 0.6)
+		(drill 0.3)
+		(layers "F.Cu" "B.Cu")
+		(free yes)
+		(net 12)
+	)
+	(via
 		(at 149.65 78.41)
 		(size 0.6)
@@
 		(polygon
 			(pts
-				(xy 107.5 100.5) (xy 107.5 106) (xy 138 106) (xy 138 100.5)
+				(xy 107.5 100.5) (xy 107.5 105.5) (xy 138 105.5) (xy 138 100.5)
 			)
 		)
@@
 		(polygon
 			(pts
-				(xy 107.5 106) (xy 107.5 111.5) (xy 138 111.5) (xy 138 106)
+				(xy 107.5 105.5) (xy 107.5 111.5) (xy 138 111.5) (xy 138 105.5)
 			)
 		)
@@
 		(polygon
 			(pts
-				(xy 116.57 75.08) (xy 150.2 75.14) (xy 150.2 94.86) (xy 116.31 95.08) (xy 116.54 75.05)
+				(xy 116.57 75.08) (xy 150.2 75.14) (xy 150.2 94.86) (xy 115.81 95.08) (xy 116.04 75.05)
 			)
 		)

Commit message: yeet
Parts:
- removed ?: , 
- BM08B-SRSS-TBLFSN1: footprint eye:CONN_BM08B-SRSS-TBLFSN_JST -> footprints:CONN_BM08B-SRSS-TBLFSN_JST
- J2: value 12V Connector -> PWM Connector
- R2: value 470 Ω -> 1000 Ω
- REF** (x2): value 6-32 -> 6 32 Hole; footprint Custom ROV Parts:6-32 -> Mounting Holes:6 32 Hole
- moved BM08B-SRSS-TBLFSN1 1.48 mm to (140.8, 80.9), turned to 0 degrees
- moved ESC5 0.09 mm to (135.0, 117.0)
- moved REF** 0.06 mm to (203.5, 81.0)
Connections:
- J2 pad 04: PWM4 -> PWM1
- J2 pad 05: Telemetry -> +5V
- J2 pad 06: PWM3 -> PWM2
- J2 pad 08: PWM2 -> PWM3
- J2 pad 09: +5V -> Telemetry
- J2 pad 10: PWM1 -> PWM4
Routing:
- net GND: track 1.19 -> 24.8 mm, vias 14 -> 12
- net PWM4: track 25.3 -> 8.22 mm, vias 2 -> 0
- net +5V: track 8.01 -> 21.6 mm, vias 0 -> 2
- net PWM1: track 12.3 -> 20.2 mm
- net PWM3: track 20.5 -> 13.0 mm
- net Telemetry: track 18.3 -> 13.2 mm, vias 2 -> 0
- net Current ADC: track 13.8 -> 17.3 mm
- net PWM2: track 16.9 -> 17.4 mm

Commit message: daniel edit for correct pwm header position + polygon adjustment
Parts:
- BM08B-SRSS-TBLFSN1: footprint footprints:CONN_BM08B-SRSS-TBLFSN_JST -> Custom:CONN_BM08B-SRSS-TBLFSN_JST
- D1: footprint led:WL-SMCW_0805 -> Diode_SMD:D_0805_2012Metric
- J2: footprint IPS1-105-01-L-D:SAMTEC_IPS1-105-01-L-D -> Custom:PWM, 12V, GND JST Connector
- R2: value 1000 Ω -> 1K Ω; footprint footprints:STA_RMCF0603_STP -> Resistor_SMD:R_0603_1608Metric
- moved BM08B-SRSS-TBLFSN1 34.6 mm to (175.3, 80.8)
- moved D1 25.9 mm to (146.4, 80.2)
- moved R2 18.2 mm to (149.4, 79.2), turned to 180 degrees
Connections:
- BM08B-SRSS-TBLFSN1 pad 1: +5V -> PWM4
- BM08B-SRSS-TBLFSN1 pad 2: GND -> PWM3
- BM08B-SRSS-TBLFSN1 pad 3: Current ADC -> PWM2
- BM08B-SRSS-TBLFSN1 pad 4: Telemetry -> PWM1
- BM08B-SRSS-TBLFSN1 pad 5: PWM1 -> +5V
- BM08B-SRSS-TBLFSN1 pad 6: PWM2 -> unconnected-(BM08B-SRSS-TBLFSN1-Pad6)
- BM08B-SRSS-TBLFSN1 pad 7: PWM3 -> GND
- BM08B-SRSS-TBLFSN1 pad 8: PWM4 -> Telemetry
- J2 pad 05: +5V -> Telemetry
- J2 pad 07: Current ADC -> unconnected-(J2-Pad07)
- J2 pad 09: Telemetry -> +5V
Routing:
- net Current ADC: track 17.3 -> 0.00 mm
- net Telemetry: track 13.2 -> 21.1 mm, vias 0 -> 2
- net +12V: track 10.1 -> 2.66 mm
- net +5V: track 21.6 -> 14.6 mm, vias 2 -> 0
- net GND: track 24.8 -> 28.5 mm, vias 12 -> 33
- net ESC2A: track 3.46 -> 0.00 mm
- net Net-(D1-Pad2): track 5.22 -> 2.20 mm
- added copper zone on F.Cu, net +12V
- added copper zone on B.Cu, net ESC1A
- added copper zone on B.Cu, net ESC1B
- added copper zone on B.Cu, net ESC1C
- added copper zone on B.Cu, net ESC2A
- added copper zone on B.Cu, net ESC2B
- added copper zone on B.Cu, net ESC2C
- added copper zone on B.Cu, net ESC3A
- added copper zone on B.Cu, net ESC3B
- added copper zone on B.Cu, net ESC3C
- added copper zone on B.Cu, net ESC4A
- added copper zone on B.Cu, net ESC4B
- added copper zone on B.Cu, net ESC4C
Other:
- board text removed: "GND"
