File: X17-ESC-Adapter/X17-ESC-Adapter.kicad_pcb (KiCad board)
At the start: 2 copper layers, 101.6 x 41.2 mm, 23 parts, among them J1 Pad for ESC, J10 Pad for ESC, J11 Pad for ESC, J12 Pad for ESC, J13 Pad for ESC, J2 PWM Connector, J3 Pad for ESC, J4 Pad for ESC, J5 Pad for ESC, J6 Pad for ESC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

Commit message: changes 1/3/25
Connections:
- BM08B-SRSS-TBLFSN1 pad 5: +5V -> Telemetry
- BM08B-SRSS-TBLFSN1 pad 8: Telemetry -> +5V
Routing:
- net Telemetry: track 21.1 -> 18.1 mm
- net +5V: track 14.6 -> 17.3 mm

Commit message: 1/10/25 gerber files
Parts:
- removed REF** (x2): 6 32 Hole, Mounting Holes:6 32 Hole
- added H1: 6-32-HOLE, X16_PowerSlab_V2:6-32-HOLE, B.Cu at (205.0, 80.5)
- added H1: 6-32-HOLE, X16_PowerSlab_V2:6-32-HOLE, B.Cu at (110.9, 80.5)
